Commit message: removed akdk_camera file in favor of lighter Azure_Kinect.stl

File: urdf/ddbot.urdf.xacro (robot description, xacro)
@@ -99,5 +99,5 @@
       <origin xyz="0 0 0" rpy="1.5707 0 1.5707" />
     <geometry>
-	      <mesh filename="package://trikey_description/meshes/akdk_camera.dae" scale="0.001 0.001 0.001"/>
+	      <mesh filename="package://trikey_description/meshes/Azure_Kinect.stl" scale="0.001 0.001 0.001"/>
       </geometry>
     </visual>
@@ -105,5 +105,5 @@
       <origin xyz="0 0 0" rpy="1.5707 0 1.5707"/>
       <geometry>
-        <mesh filename="package://trikey_description/meshes/akdk_camera.dae" scale="0.001 0.001 0.001"/>
+        <mesh filename="package://trikey_description/meshes/Azure_Kinect.stl" scale="0.001 0.001 0.001"/>
       </geometry>
     </collision>
