Commit message: urdf->xacro

File: urdf/TrikeyBaseAssembly.urdf.xacro (robot description, xacro)
@@ -1,4 +1,4 @@
-<?xml version="1.0" encoding="utf-8"?>
-<robot name="trikey">
+<?xml version="1.1"?>
+<robot name="trikey" xmlns:xacro="http://ros.org/wiki/xacro">
   <link name="base_link">
     <visual>
@@ -26,4 +26,6 @@
     </inertial>
   </link>
+  <link name= "main_body_link">
+  </link>
   <!--  Wheels  -->
   <link name="wheel0">
@@ -153,30 +155,4 @@
     </inertial>
   </link>
-  <!-- Azure Kinect Camera Link (Bottom Camera) -->
-  <link name="kinect_2_link">
-    <visual>
-      <origin xyz="0 0 0" rpy="0 0 0"/>
-      <geometry>
-        <mesh filename="package://trikey_description/meshes/Azure_Kinect.stl"/>
-      </geometry>
-      <material name="kinect_material">
-        <color rgba="0.9 0.2 0.24 1.0"/>
-      </material>
-    </visual>
-    <collision>
-      <origin xyz="0.0 0.0 0.0"/>
-      <geometry>
-        <mesh filename="package://trikey_description/meshes/Azure_Kinect.stl"/>
-      </geometry>
-      <material name="kinect_material">
-        <color rgba="0.9 0.2 0.24 1.0"/>
-      </material>
-    </collision>
-    <inertial>
-      <origin xyz="0 0 0" rpy="0 0 0"/>
-      <mass value=".44" />
-      <inertia ixx="10.173985" ixy="0.212137"  ixz="-0.09591" iyy="5.191632" iyz="0.505713" izz="5.853716" />
-    </inertial>
-  </link>
   <!-- Azure Kinect Camera Lense Link (Top Camera) -->
   <link name="kinect_1_lense_link">
@@ -188,14 +164,10 @@
     </visual>
   </link>
-  <!-- Azure Kinect Camera Lense Link (Bottom Camera) -->
-  <link name="kinect_2_lense_link">
-    <visual>
-      <origin xyz="0 0 0" rpy="0 1.57 0" />
-      <geometry>
-        <cylinder length="0.001" radius="0.01"/>
-      </geometry>
-    </visual>
-  </link>
   <!-- Joints -->
+  <joint name="main_body_joint" type="fixed">
+    <origin xyz="-0.1 -0.06 0" rpy="0 0 -1.57"/>
+    <parent link="base_link"/>
+    <child link="main_body_link"/>
+  </joint>
   <joint name="wheel0_joint" type="continuous">
     <origin xyz="-0.103157 -0.317313 -0.144393" rpy="1.5708 0.599769 -5.54919e-17" />
@@ -235,23 +207,8 @@
         <child link="camera_base"/>
     </joint>
-<!--    <joint name="kinect_1_joint" type="fixed">-->
-<!--        <origin xyz="-0.01239 -0.289682 0.28607" rpy="0 -1.0471975511965976 1.57079632679"/>-->
-<!--        <parent link="base_link"/>-->
-<!--        <child link="camera_base"/>-->
-<!--    </joint>-->
-    <joint name="kinect_2_joint" type="fixed">
-        <origin xyz="0.01239 -0.289682 0.1734" rpy="0 2.0943951023931953 -1.57079632679"/>
-        <parent link="base_link"/>
-        <child link="kinect_2_link"/>
-    </joint>
     <joint name="kinect_1_lense_joint" type="fixed">
         <origin xyz="-0.03 0 0.01" rpy="3.14 -1.57 0"/>
         <parent link="camera_base"/>
         <child link="kinect_1_lense_link"/>
-    </joint>
-    <joint name="kinect_2_lense_joint" type="fixed">
-        <origin xyz="-0.03 0 0.01" rpy="0 -1.57 0"/>
-        <parent link="kinect_2_link"/>
-        <child link="kinect_2_lense_link"/>
     </joint>
   <!-- Camera Plugin for Gazebo -->
@@ -298,41 +255,4 @@
       </sensor>
     </gazebo>
-    <!-- Kinect Camera 2 -->
-    <gazebo reference="kinect_2_lense_link">
-      <sensor type="depth" name="camera2">
-        <update_rate>15.0</update_rate>
-        <camera name="kinect2">
-          <horizontal_fov>2.0944</horizontal_fov>
-          <image>
-            <width>512</width>
-            <height>512</height>
-            <format>R8G8B8</format>
-          </image>
-          <clip>
-            <near>0.02</near>
-            <far>300</far>
-          </clip>
-          <noise>
-            <type>gaussian</type>
-            <mean>0.5</mean>
-            <stddev>0.007</stddev>
-          </noise>
-        </camera>
-          <plugin name="kinect_plugin" filename="libgazebo_ros_openni_kinect.so">
-                <baseline>0.1</baseline>
-                <alwaysOn>true</alwaysOn>
-                <updateRate>0.0</updateRate>
-                <cameraName>kinect2</cameraName>
-                <imageTopicName>/kinect2/color/image_raw</imageTopicName>
-                <cameraInfoTopicName>/kinect2/camera_info</cameraInfoTopicName>
-                <depthImageTopicName>/kinect2/depth/image_raw</depthImageTopicName>
-                <depthImageInfoTopicName>/kinect2/depth/camera_info</depthImageInfoTopicName>
-                <pointCloudTopicName>/kinect2/points</pointCloudTopicName>
-                <frameName>kinect_2_lense_link</frameName>
-                <pointCloudCutoff>0.5</pointCloudCutoff>
-                <pointCloudCutoffMax>2.0</pointCloudCutoffMax>
-            </plugin>
-      </sensor>
-    </gazebo>
   <!-- Transmissions: needed for ROS control -->
   <transmission name="wheel0_simple_trans">

Commit message: TirkeyBaseAssembly Xacro conversion

File: urdf/TrikeyBaseAssembly.urdf.xacro (robot description, xacro)
@@ -1,5 +1,9 @@
 <?xml version="1.1"?>
 <robot name="trikey" xmlns:xacro="http://ros.org/wiki/xacro">
-  <link name="base_link">
+<!-- Include Gazebo plugins -->
+<xacro:include filename="$(find trikey_description)/urdf/urdf_gazebo/robot.gazebo.xacro" />
+  <link name= "base_link">
+  </link>
+  <link name="body_link">
     <visual>
       <origin xyz="0.00252107 -0.0402364 -0.0133064" rpy="0 -0 0" />
@@ -26,6 +30,4 @@
     </inertial>
   </link>
-  <link name= "main_body_link">
-  </link>
   <!--  Wheels  -->
   <link name="wheel0">
@@ -130,5 +132,5 @@
   </link>
   <!-- Azure Kinect Camera Link (Top Camera) -->
-  <link name="camera_base">
+  <link name="camera_link">
     <visual>
       <origin xyz="0 0 0" rpy="0 0 0"/>
@@ -165,12 +167,12 @@
   </link>
   <!-- Joints -->
-  <joint name="main_body_joint" type="fixed">
-    <origin xyz="-0.1 -0.06 0" rpy="0 0 -1.57"/>
+  <joint name="body_joint" type="fixed">
+    <origin xyz="-0.06 0.1 0" rpy="0 0 1.57"/>
     <parent link="base_link"/>
-    <child link="main_body_link"/>
+    <child link="body_link"/>
   </joint>
   <joint name="wheel0_joint" type="continuous">
     <origin xyz="-0.103157 -0.317313 -0.144393" rpy="1.5708 0.599769 -5.54919e-17" />
-    <parent link="base_link" />
+    <parent link="body_link" />
     <child link="wheel0" />
     <axis xyz="0 0 1"/>
@@ -180,5 +182,5 @@
   <joint name="wheel1_joint" type="continuous">
     <origin xyz="0.110261 0.0612702 -0.144393" rpy="1.5708 0.632117 2.0944" />
-    <parent link="base_link" />
+    <parent link="body_link" />
     <child link="wheel1" />
     <axis xyz="0 0 1"/>
@@ -188,5 +190,5 @@
   <joint name="wheel2_joint" type="continuous">
     <origin xyz="-0.323445 0.0653045 -0.144393" rpy="-1.5708 -1.38778e-17 1.0472" />
-    <parent link="base_link" />
+    <parent link="body_link" />
     <child link="wheel2" />
     <axis xyz="0 0 1"/>
@@ -198,5 +200,5 @@
   <joint name="lidar_joint" type="fixed">
     <origin xyz="-0.103 -0.289682 0.34108" rpy="0. 0. 1.57079632"/>
-    <parent link="base_link"/>
+    <parent link="body_link"/>
     <child link="lidar_link"/>
   </joint>
@@ -204,121 +206,11 @@
     <joint name="kinect_1_joint" type="fixed">
         <origin xyz="-0.1144 -0.261352 0.22108" rpy="0 -1.57079632679 1.57079632679"/>
-        <parent link="base_link"/>
-        <child link="camera_base"/>
+        <parent link="body_link"/>
+        <child link="camera_link"/>
     </joint>
     <joint name="kinect_1_lense_joint" type="fixed">
         <origin xyz="-0.03 0 0.01" rpy="3.14 -1.57 0"/>
-        <parent link="camera_base"/>
+        <parent link="camera_link"/>
         <child link="kinect_1_lense_link"/>
     </joint>
-  <!-- Camera Plugin for Gazebo -->
-  <!-- Note on gaussian noise statistics:
-  Noise is sampled independently per pixel on each frame. That pixel's noise value is added
-  to each of its color channels, which at that point lie in the range [0,1]. -->
-  <!-- Note on kinect plugin:
-  Keep update_rate to zero, update_rate in the parent <sensor> tag will control the frame rate. -->
-  <!-- Kinect Camera 1 -->
-    <gazebo reference="kinect_1_lense_link">
-      <sensor type="depth" name="camera1">
-        <update_rate>15.0</update_rate>
-        <camera name="kinect1">
-          <horizontal_fov>2.0944</horizontal_fov>
-          <image>
-            <width>512</width>
-            <height>512</height>
-            <format>R8G8B8</format>
-          </image>
-          <clip>
-            <near>0.02</near>
-            <far>300</far>
-          </clip>
-          <noise>
-            <type>gaussian</type>
-            <mean>0.5</mean>
-            <stddev>0.007</stddev>
-          </noise>
-        </camera>
-          <plugin name="kinect_plugin" filename="libgazebo_ros_openni_kinect.so">
-                <baseline>0.1</baseline>
-                <alwaysOn>true</alwaysOn>
-                <updateRate>0.0</updateRate>
-                <cameraName>kinect1</cameraName>
-                <imageTopicName>/kinect1/color/image_raw</imageTopicName>
-                <cameraInfoTopicName>/kinect1/camera_info</cameraInfoTopicName>
-                <depthImageTopicName>/kinect1/depth/image_raw</depthImageTopicName>
-                <depthImageInfoTopicName>/kinect1/depth/camera_info</depthImageInfoTopicName>
-                <pointCloudTopicName>/kinect1/points</pointCloudTopicName>
-                <frameName>kinect_1_lense_link</frameName>
-                <pointCloudCutoff>0.5</pointCloudCutoff>
-                <pointCloudCutoffMax>2.0</pointCloudCutoffMax>
-            </plugin>
-      </sensor>
-    </gazebo>
-  <!-- Transmissions: needed for ROS control -->
-  <transmission name="wheel0_simple_trans">
-    <type>transmission_interface/SimpleTransmission</type>
-    <joint name="wheel0_joint">
-      <hardwareInterface>hardware_interface/EffortJointInterface</hardwareInterface>
-    </joint>
-    <actuator name="wheel0_motor">
-      <hardwareInterface>hardware_interface/EffortJointInterface</hardwareInterface>
-    </actuator>
-  </transmission>
-  <transmission name="wheel1_simple_trans">
-    <type>transmission_interface/SimpleTransmission</type>
-    <joint name="wheel1_joint">
-      <hardwareInterface>hardware_interface/EffortJointInterface</hardwareInterface>
-    </joint>
-    <actuator name="wheel1_motor">
-      <hardwareInterface>hardware_interface/EffortJointInterface</hardwareInterface>
-    </actuator>
-  </transmission>
-  <transmission name="wheel2_simple_trans">
-    <type>transmission_interface/SimpleTransmission</type>
-    <joint name="wheel2_joint">
-      <hardwareInterface>hardware_interface/EffortJointInterface</hardwareInterface>
-    </joint>
-    <actuator name="wheel2_motor">
-      <hardwareInterface>hardware_interface/EffortJointInterface</hardwareInterface>
-    </actuator>
-  </transmission>
-  <!-- Sensors -->
-  <!--
-  <gazebo reference="lidar_link">
-    <sensor type="ray" name="rplidar">
-      <pose>0 0 0 0 0 0</pose>
-      <visualize>true</visualize>
-      <update_rate>10</update_rate>
-      <ray>
-        <scan>
-          <horizontal>
-            <samples>400</samples>
-            <resolution>1</resolution>
-	    <min_angle>-3.141592</min_angle>
-            <max_angle>3.141592 </max_angle>
-          </horizontal>
-        </scan>
-        <range>
-          <min>0.15</min>
-          <max>8.0</max>
-          <resolution>0.01</resolution>
-        </range>
-        <noise>
-          <type>gaussian</type>
-          <mean>0.0</mean>
-          <stddev>0.01</stddev>
-        </noise>
-      </ray>
-      <plugin name="gazebo_ros_lidar_controller" filename="libgazebo_ros_laser.so">
-        <topicName>/scan</topicName>
-        <frameName>base_link</frameName>
-      </plugin>
-    </sensor>
-  </gazebo>
- -->
-  <gazebo>
-    <plugin name="gazebo_ros_control" filename="libgazebo_ros_control.so">
-      <robotNamespace>/trikey</robotNamespace>
-    </plugin>
-  </gazebo>
 </robot>

File: urdf/urdf_gazebo/robot.urdf.xacro (robot description, xacro)
@@ -1,5 +1,4 @@
 <?xml version="1.1"?>
 <robot name="trikey" xmlns:xacro="http://ros.org/wiki/xacro">
- <xacro:include filename="$(find trikey_description)/urdf/urdf_gazebo/robot.gazebo.xacro" />
   <link name="base_link">
     <visual>

Commit message: urdf y faces camera

File: urdf/TrikeyBaseAssembly.urdf.xacro (robot description, xacro)
@@ -31,5 +31,5 @@
   </link>
   <!--  Wheels  -->
-  <link name="wheel0">
+  <link name="wheel2">
     <visual>
       <origin xyz="0.0157175 -0.000676884 -0.0110091" rpy="-1.5708 -3.56009e-33 -5.76344e-17" />
@@ -56,5 +56,5 @@
     </inertial>
   </link>
-  <link name="wheel1">
+  <link name="wheel0">
     <visual>
       <origin xyz="0.0157175 -0.000676884 -0.0110091" rpy="-1.5708 4.8608e-17 1.36846e-47" />
@@ -81,5 +81,5 @@
     </inertial>
   </link>
-  <link name="wheel2">
+  <link name="wheel1">
     <visual>
       <origin xyz="0.0157175 -0.000676884 -0.00283407" rpy="-1.5708 -2.51863e-17 3.13582e-17" />
@@ -168,10 +168,18 @@
   <!-- Joints -->
   <joint name="body_joint" type="fixed">
-    <origin xyz="-0.06 0.1 0" rpy="0 0 1.57"/>
+    <origin xyz="-0.1 -0.06 0" rpy="0 0 3.14"/>
     <parent link="base_link"/>
     <child link="body_link"/>
   </joint>
+  <joint name="wheel2_joint" type="continuous">
+    <origin xyz="-0.103157 -0.317313 -0.144393" rpy="1.5708 0.599769 -5.54919e-17" />
+    <parent link="body_link" />
+    <child link="wheel2" />
+    <axis xyz="0 0 1"/>
+    <limit effort="2" velocity="20" />
+    <joint_properties friction="0.0"/>
+  </joint>
   <joint name="wheel0_joint" type="continuous">
-    <origin xyz="-0.103157 -0.317313 -0.144393" rpy="1.5708 0.599769 -5.54919e-17" />
+    <origin xyz="0.110261 0.0612702 -0.144393" rpy="1.5708 0.632117 2.0944" />
     <parent link="body_link" />
     <child link="wheel0" />
@@ -181,15 +189,7 @@
   </joint>
   <joint name="wheel1_joint" type="continuous">
-    <origin xyz="0.110261 0.0612702 -0.144393" rpy="1.5708 0.632117 2.0944" />
+    <origin xyz="-0.323445 0.0653045 -0.144393" rpy="-1.5708 -1.38778e-17 1.0472" />
     <parent link="body_link" />
     <child link="wheel1" />
-    <axis xyz="0 0 1"/>
-    <limit effort="2" velocity="20" />
-    <joint_properties friction="0.0"/>
-  </joint>
-  <joint name="wheel2_joint" type="continuous">
-    <origin xyz="-0.323445 0.0653045 -0.144393" rpy="-1.5708 -1.38778e-17 1.0472" />
-    <parent link="body_link" />
-    <child link="wheel2" />
     <axis xyz="0 0 1"/>
     <limit effort="2" velocity="20" />

Commit message: Revert "urdf y faces camera"
This reverts commit 9bc8a15cdbdef180e0a0c6d11148f10dff626fe3.

File: urdf/TrikeyBaseAssembly.urdf.xacro (robot description, xacro)
@@ -31,5 +31,5 @@
   </link>
   <!--  Wheels  -->
-  <link name="wheel2">
+  <link name="wheel0">
     <visual>
       <origin xyz="0.0157175 -0.000676884 -0.0110091" rpy="-1.5708 -3.56009e-33 -5.76344e-17" />
@@ -56,5 +56,5 @@
     </inertial>
   </link>
-  <link name="wheel0">
+  <link name="wheel1">
     <visual>
       <origin xyz="0.0157175 -0.000676884 -0.0110091" rpy="-1.5708 4.8608e-17 1.36846e-47" />
@@ -81,5 +81,5 @@
     </inertial>
   </link>
-  <link name="wheel1">
+  <link name="wheel2">
     <visual>
       <origin xyz="0.0157175 -0.000676884 -0.00283407" rpy="-1.5708 -2.51863e-17 3.13582e-17" />
@@ -168,18 +168,10 @@
   <!-- Joints -->
   <joint name="body_joint" type="fixed">
-    <origin xyz="-0.1 -0.06 0" rpy="0 0 3.14"/>
+    <origin xyz="-0.06 0.1 0" rpy="0 0 1.57"/>
     <parent link="base_link"/>
     <child link="body_link"/>
   </joint>
-  <joint name="wheel2_joint" type="continuous">
+  <joint name="wheel0_joint" type="continuous">
     <origin xyz="-0.103157 -0.317313 -0.144393" rpy="1.5708 0.599769 -5.54919e-17" />
-    <parent link="body_link" />
-    <child link="wheel2" />
-    <axis xyz="0 0 1"/>
-    <limit effort="2" velocity="20" />
-    <joint_properties friction="0.0"/>
-  </joint>
-  <joint name="wheel0_joint" type="continuous">
-    <origin xyz="0.110261 0.0612702 -0.144393" rpy="1.5708 0.632117 2.0944" />
     <parent link="body_link" />
     <child link="wheel0" />
@@ -189,7 +181,15 @@
   </joint>
   <joint name="wheel1_joint" type="continuous">
+    <origin xyz="0.110261 0.0612702 -0.144393" rpy="1.5708 0.632117 2.0944" />
+    <parent link="body_link" />
+    <child link="wheel1" />
+    <axis xyz="0 0 1"/>
+    <limit effort="2" velocity="20" />
+    <joint_properties friction="0.0"/>
+  </joint>
+  <joint name="wheel2_joint" type="continuous">
     <origin xyz="-0.323445 0.0653045 -0.144393" rpy="-1.5708 -1.38778e-17 1.0472" />
     <parent link="body_link" />
-    <child link="wheel1" />
+    <child link="wheel2" />
     <axis xyz="0 0 1"/>
     <limit effort="2" velocity="20" />

Commit message: moved lidar to wheel 2

File: urdf/TrikeyBaseAssembly.urdf.xacro (robot description, xacro)
@@ -199,6 +199,6 @@
   <!-- distance from chassis STL origin to actual center (manually tuned): [-0.103 -0.057 0] -->
   <joint name="lidar_joint" type="fixed">
-    <origin xyz="-0.103 -0.289682 0.34108" rpy="0. 0. 1.57079632"/>
-    <parent link="body_link"/>
+    <origin xyz="-0.136 -0.2355 0.34108" rpy="0. 0. 1.57079632"/>
+    <parent link="base_link"/>
     <child link="lidar_link"/>
   </joint>
