Commit message: urdf -> urdf.xacro

File: urdf/urdf_generator/robot.urdf.xacro (robot description, xacro)
@@ -1,10 +1,4 @@
-<robot name="trikey">
-    <!-- <link name="odom"/> -->
-<!--
-    <joint name="floating_base_joint" type="fixed">
-        <origin xyz="0 0 0.0" rpy="0 0 0"/>
-        <parent link="odom"/>
-        <child link="base_link"/>
-    </joint> -->
+<?xml version="1.1"?>
+<robot name="trikey" xmlns:xacro="http://ros.org/wiki/xacro">
 <link name="base_link">
 <visual>
@@ -2031,5 +2025,5 @@
     <!-- Kinect Camera Joints -->
     <joint name="kinect_1_joint" type="fixed">
-        <origin xyz="-0.01239 -0.289682 0.28607" rpy="0 -1.0471975511965976 1.57079632679"/>
+        <origin xyz="-0.01239 -0.289682 0.28607" rpy="0 1.57 -1.57079632679"/>
         <parent link="base_link"/>
         <child link="kinect_1_link"/>

Commit message: robot-> robot.urdf.xacro & robot.gazebo.xacro

File: urdf/urdf_generator/robot.urdf.xacro (robot description, xacro)
@@ -1,5 +1,13 @@
 <?xml version="1.1"?>
 <robot name="trikey" xmlns:xacro="http://ros.org/wiki/xacro">
-<link name="base_link">
+<xacro:include filename="$(find trikey_description)/urdf/urdf_generator/robot.gazebo.xacro" />
+<link name= "base_link">
+</link>
+<joint name="body_joint" type="fixed">
+    <origin xyz="0 0 0" rpy="0 0 3.14"/>
+    <parent link="base_link"/>
+    <child link="body_link"/>
+</joint>
+<link name="body_link">
 <visual>
 <origin xyz="0.007652 0.00490494 0.000231732" rpy="-1.11735e-06 1.93532e-06 2.69365e-06" />
@@ -647,5 +655,5 @@
 <joint name="wheel0_joint" type="continuous">
 <origin xyz="0.0076339 -0.242491 -0.130854" rpy="1.5708 1.50474e-12 2.69365e-06" />
-<parent link="base_link" />
+<parent link="body_link" />
 <child link="wheel" />
 <axis xyz="0 0 1"/>
@@ -1274,5 +1282,5 @@
 <joint name="wheel1_joint" type="continuous">
 <origin xyz="-0.212654 0.132125 -0.130854" rpy="-1.5708 -1.50485e-12 1.0472" />
-<parent link="base_link" />
+<parent link="body_link" />
 <child link="wheel_2" />
 <axis xyz="0 0 1"/>
@@ -1901,5 +1909,5 @@
 <joint name="wheel2_joint" type="continuous">
 <origin xyz="0.227979 0.132092 -0.130855" rpy="-1.5708 -3.25141e-07 -1.04719" />
-<parent link="base_link" />
+<parent link="body_link" />
 <child link="wheel_3" />
 <axis xyz="0 0 1"/>
@@ -1922,5 +1930,5 @@
     <joint name="lidar_mount_joint" type="fixed">
         <origin xyz="0.0 -0.23 0.345" rpy="0.0 0.0 0.0"/>
-        <parent link="base_link"/>
+        <parent link="body_link"/>
         <child link="lidar_mount"/>
     </joint>
@@ -1972,5 +1980,5 @@
     </link>
     <!-- Azure Kinect Camera Link (Bottom Camera) -->
-    <link name="kinect_2_link">
+    <!-- <link name="kinect_2_link">
         <visual>
             <origin xyz="0 0 0" rpy="0 0 0"/>
@@ -1996,5 +2004,5 @@
             <inertia ixx="10.173985" ixy="0.212137"  ixz="-0.09591" iyy="5.191632" iyz="0.505713" izz="5.853716" />
         </inertial>
-    </link>
+    </link> -->
   <!-- Azure Kinect Camera Lense Link (Top Camera) -->
   <link name="kinect_1_lense_link">
@@ -2007,5 +2015,5 @@
   </link>
   <!-- Azure Kinect Camera Lense Link (Bottom Camera) -->
-  <link name="kinect_2_lense_link">
+  <!-- <link name="kinect_2_lense_link">
     <visual>
       <origin xyz="0 0 0" rpy="0 1.57 0" />
@@ -2022,16 +2030,16 @@
       </geometry>
     </visual>
-  </link>
+  </link> -->
     <!-- Kinect Camera Joints -->
     <joint name="kinect_1_joint" type="fixed">
         <origin xyz="-0.01239 -0.289682 0.28607" rpy="0 1.57 -1.57079632679"/>
-        <parent link="base_link"/>
+        <parent link="body_link"/>
         <child link="kinect_1_link"/>
     </joint>
-    <joint name="kinect_2_joint" type="fixed">
+    <!-- <joint name="kinect_2_joint" type="fixed">
         <origin xyz="0.01239 -0.289682 0.1734" rpy="0 2.0943951023931953 -1.57079632679"/>
-        <parent link="base_link"/>
+        <parent link="body_link"/>
         <child link="kinect_2_link"/>
-    </joint>
+    </joint> -->
     <joint name="kinect_1_lense_joint" type="fixed">
         <origin xyz="-0.03 0 0.01" rpy="3.14 -1.57 0"/>
@@ -2039,5 +2047,5 @@
         <child link="kinect_1_lense_link"/>
     </joint>
-    <joint name="kinect_2_lense_joint" type="fixed">
+    <!-- <joint name="kinect_2_lense_joint" type="fixed">
         <origin xyz="-0.03 0 0.01" rpy="0 -1.57 0"/>
         <parent link="kinect_2_link"/>
@@ -2048,5 +2056,5 @@
         <parent link="kinect_2_link"/>
         <child link="kinect_2_pcl_link"/>
-    </joint>
+    </joint> -->
     <!-- Lidar Joint -->
     <joint name="rplidar_joint" type="fixed">
@@ -2056,610 +2064,3 @@
         <child link="rplidar_link"/>
     </joint>
-    <!-- RPLidar Sensor -->
-    <!-- Noise parameters based on published spec for Hokuyo laser
-    achieving "+-30mm" accuracy at range < 10m.  A mean of 0.0m and
-    stddev of 0.01m will put 99.7% of samples within 0.03m of the true
-    reading. -->
-    <!-- specs for RPLidar A2M8
-    <gazebo reference="rplidar_link">
-        <sensor type="ray" name="rplidar_sensor">
-          <pose>0 0 1 0 0 0</pose>
-          <visualize>true</visualize>
-          <update_rate>10</update_rate>
-          <ray>
-            <scan>
-              <horizontal>
-                <samples>400</samples>
-                <resolution>1</resolution>
-                <min_angle>-3.141593</min_angle>
-                <max_angle>3.141593</max_angle>
-              </horizontal>
-	    </scan>
-            <range>
-              <min>0.15</min>
-              <max>8.0</max>
-              <resolution>0.01</resolution>
-            </range>
-            <noise>
-              <type>gaussian</type>
-               <mean>0.0</mean>
-              <stddev>0.01</stddev>
-            </noise>
-          </ray>
-            <plugin name="gazebo_ros_head_rplidar_controller" filename="libgazebo_ros_laser.so">
-            <topicName>/scan</topicName>
-            <frameName>rplidar_link</frameName>
-        </plugin>
-        </sensor>
-        <material>Gazebo/Grey</material>
-     </gazebo>
-     -->
-  <!-- Camera Plugin for Gazebo -->
-    <!-- Kinect Camera 1 -->
-    <gazebo reference="kinect_1_lense_link">
-      <sensor type="depth" name="camera1">
-        <update_rate>15.0</update_rate>
-        <camera name="kinect1">
-          <horizontal_fov>2.0944</horizontal_fov>
-          <image>
-            <width>512</width>
-            <height>512</height>
-            <format>R8G8B8</format>
-          </image>
-          <clip>
-            <near>0.02</near>
-            <far>300</far>
-          </clip>
-          <noise>
-            <type>gaussian</type>
-            <!-- Noise is sampled independently per pixel on each frame.
-                That pixel's noise value is added to each of its color
-                channels, which at that point lie in the range [0,1]. -->
-            <mean>0.5</mean>
-            <stddev>0.007</stddev>
-          </noise>
-        </camera>
-          <plugin name="kinect_plugin" filename="libgazebo_ros_openni_kinect.so">
-                <baseline>0.1</baseline>
-                <alwaysOn>true</alwaysOn>
-                <!-- Keep this zero, update_rate in the parent <sensor> tag
-                will control the frame rate. -->
-                <updateRate>0.0</updateRate>
-                <cameraName>kinect1</cameraName>
-                <robotNamespace>/trikey</robotNamespace>
-                <imageTopicName>/kinect1/color/image_raw</imageTopicName>
-                <cameraInfoTopicName>/kinect1/camera_info</cameraInfoTopicName>
-                <depthImageTopicName>/kinect1/depth/image_raw</depthImageTopicName>
-                <depthImageInfoTopicName>/kinect1/depth/camera_info</depthImageInfoTopicName>
-                <pointCloudTopicName>/kinect1/points</pointCloudTopicName>
-                <frameName>kinect_1_lense_link</frameName>
-                <pointCloudCutoff>0.5</pointCloudCutoff>
-                <pointCloudCutoffMax>2.0</pointCloudCutoffMax>
-            </plugin>
-      </sensor>
-    </gazebo>
-    <!-- Kinect Camera 2 -->
-    <gazebo reference="kinect_2_lense_link">
-      <sensor type="depth" name="camera2">
-        <update_rate>15.0</update_rate>
-        <camera name="kinect2">
-          <horizontal_fov>2.0944</horizontal_fov>
-          <image>
-            <width>512</width>
-            <height>512</height>
-            <format>R8G8B8</format>
-          </image>
-          <clip>
-            <near>0.02</near>
-            <far>300</far>
-          </clip>
-          <noise>
-            <type>gaussian</type>
-            <!-- Noise is sampled independently per pixel on each frame.
-                That pixel's noise value is added to each of its color
-                channels, which at that point lie in the range [0,1]. -->
-            <mean>0.5</mean>
-            <stddev>0.007</stddev>
-          </noise>
-        </camera>
-          <plugin name="kinect_plugin" filename="libgazebo_ros_openni_kinect.so">
-                <baseline>0.1</baseline>
-                <alwaysOn>true</alwaysOn>
-                <!-- Keep this zero, update_rate in the parent <sensor> tag
-                will control the frame rate. -->
-                <updateRate>0.0</updateRate>
-                <cameraName>kinect2</cameraName>
-                <robotNamespace>/trikey</robotNamespace>
-                <imageTopicName>/kinect2/color/image_raw</imageTopicName>
-                <cameraInfoTopicName>/kinect2/camera_info</cameraInfoTopicName>
-                <depthImageTopicName>/kinect2/depth/image_raw</depthImageTopicName>
-                <depthImageInfoTopicName>/kinect2/depth/camera_info</depthImageInfoTopicName>
-                <pointCloudTopicName>/kinect2/points</pointCloudTopicName>
-                <frameName>kinect_2_pcl_link</frameName>
-                <pointCloudCutoff>0.5</pointCloudCutoff>
-                <pointCloudCutoffMax>2.0</pointCloudCutoffMax>
-            </plugin>
-      </sensor>
-    </gazebo>
-    <!-- Transmissions: needed for ROS control -->
-    <transmission name="wheel0_simple_trans">
-        <type>transmission_interface/SimpleTransmission</type>
-        <joint name="wheel0_joint">
-            <hardwareInterface>hardware_interface/EffortJointInterface</hardwareInterface>
-        </joint>
-        <actuator name="wheel0_motor">
-            <hardwareInterface>hardware_interface/EffortJointInterface</hardwareInterface>
-        </actuator>
-    </transmission>
-    <transmission name="wheel1_simple_trans">
-        <type>transmission_interface/SimpleTransmission</type>
-        <joint name="wheel1_joint">
-            <hardwareInterface>hardware_interface/EffortJointInterface</hardwareInterface>
-        </joint>
-        <actuator name="wheel1_motor">
-            <hardwareInterface>hardware_interface/EffortJointInterface</hardwareInterface>
-        </actuator>
-    </transmission>
-    <transmission name="wheel2_simple_trans">
-        <type>transmission_interface/SimpleTransmission</type>
-        <joint name="wheel2_joint">
-            <hardwareInterface>hardware_interface/EffortJointInterface</hardwareInterface>
-        </joint>
-        <actuator name="wheel2_motor">
-            <hardwareInterface>hardware_interface/EffortJointInterface</hardwareInterface>
-        </actuator>
-    </transmission>
-    <!--==================== Sensors ====================-->
-    <!-- Pose Ground Truth -->
-    <gazebo>
-        <plugin filename="libgazebo_ros_p3d.so" name="gazebo_ros_p3d">
-            <robotNamespace>/trikey</robotNamespace>
-            <frame_name>odom</frame_name>
-            <bodyName>base_link</bodyName>
-            <topicName>ground_truth</topicName>
-            <frameName>world</frameName>
-            <gaussianNoise>0</gaussianNoise>
-            <alwaysOn>true</alwaysOn>
-            <updateRate>30</updateRate>
-        </plugin>
-    </gazebo>
-    <gazebo>
-        <plugin name="gazebo_ros_control" filename="libgazebo_ros_control.so">
-            <robotNamespace>/trikey</robotNamespace>
-            <controlPeriod>0.001</controlPeriod>
-        </plugin>
-    </gazebo>
-    <!-- Fix jitter -->
-    <gazebo reference="8x750roller">
-        <mu1>0.8</mu1>
-        <mu2>0.8</mu2>
-        <kp>50000.0</kp>
-        <kd>80.0</kd>
-        <minDepth>0.0001</minDepth>
-        <maxVel>0</maxVel>
-    </gazebo>
-    <gazebo reference="8x750roller_2">
-        <mu1>0.8</mu1>
-        <mu2>0.8</mu2>
-        <kp>50000.0</kp>
-        <kd>80.0</kd>
-        <minDepth>0.0001</minDepth>
-        <maxVel>0</maxVel>
-    </gazebo>
-    <gazebo reference="8x750roller_3">
-        <mu1>0.8</mu1>
-        <mu2>0.8</mu2>
-        <kp>50000.0</kp>
-        <kd>80.0</kd>
-        <minDepth>0.0001</minDepth>
-        <maxVel>0</maxVel>
-    </gazebo>
-    <gazebo reference="8x750roller_4">
-        <mu1>0.8</mu1>
-        <mu2>0.8</mu2>
-        <kp>50000.0</kp>
-        <kd>80.0</kd>
-        <minDepth>0.0001</minDepth>
-        <maxVel>0</maxVel>
-    </gazebo>
-    <gazebo reference="8x750roller_5">
-        <mu1>0.8</mu1>
-        <mu2>0.8</mu2>
-        <kp>50000.0</kp>
-        <kd>80.0</kd>
-        <minDepth>0.0001</minDepth>
-        <maxVel>0</maxVel>
-    </gazebo>
-    <gazebo reference="8x750roller_6">
-        <mu1>0.8</mu1>
-        <mu2>0.8</mu2>
-        <kp>50000.0</kp>
-        <kd>80.0</kd>
-        <minDepth>0.0001</minDepth>
-        <maxVel>0</maxVel>
-    </gazebo>
-    <gazebo reference="8x750roller_7">
-        <mu1>0.8</mu1>
-        <mu2>0.8</mu2>
-        <kp>50000.0</kp>
-        <kd>80.0</kd>
-        <minDepth>0.0001</minDepth>
-        <maxVel>0</maxVel>
-    </gazebo>
-    <gazebo reference="8x750roller_8">
-        <mu1>0.8</mu1>
-        <mu2>0.8</mu2>
-        <kp>50000.0</kp>
-        <kd>80.0</kd>
-        <minDepth>0.0001</minDepth>
-        <maxVel>0</maxVel>
-    </gazebo>
-    <gazebo reference="8x750roller_9">
-        <mu1>0.8</mu1>
-        <mu2>0.8</mu2>
-        <kp>50000.0</kp>
-        <kd>80.0</kd>
-        <minDepth>0.0001</minDepth>
-        <maxVel>0</maxVel>
-    </gazebo>
-    <gazebo reference="8x750roller_10">
-        <mu1>0.8</mu1>
-        <mu2>0.8</mu2>
-        <kp>50000.0</kp>
-        <kd>80.0</kd>
-        <minDepth>0.0001</minDepth>
-        <maxVel>0</maxVel>
-    </gazebo>
-    <gazebo reference="8x750roller_11">
-        <mu1>0.8</mu1>
-        <mu2>0.8</mu2>
-        <kp>50000.0</kp>
-        <kd>80.0</kd>
-        <minDepth>0.0001</minDepth>
-        <maxVel>0</maxVel>
-    </gazebo>
-    <gazebo reference="8x750roller_12">
-        <mu1>0.8</mu1>
-        <mu2>0.8</mu2>
-        <kp>50000.0</kp>
-        <kd>80.0</kd>
-        <minDepth>0.0001</minDepth>
-        <maxVel>0</maxVel>
-    </gazebo>
-    <gazebo reference="8x750roller_13">
-        <mu1>0.8</mu1>
-        <mu2>0.8</mu2>
-        <kp>50000.0</kp>
-        <kd>80.0</kd>
-        <minDepth>0.0001</minDepth>
-        <maxVel>0</maxVel>
-    </gazebo>
-    <gazebo reference="8x750roller_14">
-        <mu1>0.8</mu1>
-        <mu2>0.8</mu2>
-        <kp>50000.0</kp>
-        <kd>80.0</kd>
-        <minDepth>0.0001</minDepth>
-        <maxVel>0</maxVel>
-    </gazebo>
-    <gazebo reference="8x750roller_15">
-        <mu1>0.8</mu1>
-        <mu2>0.8</mu2>
-        <kp>50000.0</kp>
-        <kd>80.0</kd>
-        <minDepth>0.0001</minDepth>
-        <maxVel>0</maxVel>
-    </gazebo>
-    <gazebo reference="8x750roller_16">
-        <mu1>0.8</mu1>
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
Commit message: started fixing coord frame in rviz

File: urdf/urdf_generator/robot.urdf.xacro (robot description, xacro)
@@ -1921,5 +1921,5 @@
     </link>
     <joint name="lidar_mount_joint" type="fixed">
-        <origin xyz="0.0 -0.23 0.345" rpy="0.0 0.0 0.0"/>
+        <origin xyz="-0.2355 0.136 0.345" rpy="0.0 0.0 0.0"/>
         <parent link="base_link"/>
         <child link="lidar_mount"/>
