Commit message: wheel1,2,3 -> wheel0,1,2

File: urdf/urdf_generator/robot.urdf.xacro (robot description, xacro)
@@ -34,5 +34,5 @@
 </inertial>
 </link>
-<link name="wheel">
+<link name="wheel0">
 <visual>
 <origin xyz="0.0157175 -0.000676884 -0.00283407" rpy="-1.5708 1.4944e-22 -1.48983e-28" />
@@ -86,5 +86,5 @@
 <joint name="roller_w0_0" type="continuous">
 <origin xyz="0.0835653 -0.0394107 0.0065875" rpy="-1.5708 1.57079 -0.523599" />
-<parent link="wheel" />
+<parent link="wheel0" />
 <child link="8x750roller" />
 <axis xyz="0 0 1"/>
@@ -119,5 +119,5 @@
 <joint name="roller_w0_1" type="continuous">
 <origin xyz="0.0665785 -0.0643294 0.0065875" rpy="-0.698132 1.5708 0" />
-<parent link="wheel" />
+<parent link="wheel0" />
 <child link="8x750roller_2" />
 <axis xyz="0 0 1"/>
@@ -152,5 +152,5 @@
 <joint name="roller_w0_2" type="continuous">
 <origin xyz="0.0405614 -0.083221 0.0065875" rpy="-0.349066 1.5708 0" />
-<parent link="wheel" />
+<parent link="wheel0" />
 <child link="8x750roller_3" />
 <axis xyz="0 0 1"/>
@@ -185,5 +185,5 @@
 <joint name="roller_w0_3" type="continuous">
 <origin xyz="0.009652 -0.092075 0.0065875" rpy="1.5708 1.5708 1.5708" />
-<parent link="wheel" />
+<parent link="wheel0" />
 <child link="8x750roller_4" />
 <axis xyz="0 0 1"/>
@@ -218,5 +218,5 @@
 <joint name="roller_w0_4" type="continuous">
 <origin xyz="-0.0224216 -0.0898234 0.0065875" rpy="1.5708 1.57079 1.22173" />
-<parent link="wheel" />
+<parent link="wheel0" />
 <child link="8x750roller_5" />
 <axis xyz="0 0 1"/>
@@ -251,5 +251,5 @@
 <joint name="roller_w0_5" type="continuous">
 <origin xyz="-0.0517908 -0.0767377 0.0065875" rpy="1.5708 1.57079 0.872665" />
-<parent link="wheel" />
+<parent link="wheel0" />
 <child link="8x750roller_6" />
 <axis xyz="0 0 1"/>
@@ -284,5 +284,5 @@
 <joint name="roller_w0_6" type="continuous">
 <origin xyz="-0.0749133 -0.0543964 0.0065875" rpy="1.5708 1.57079 0.523599" />
-<parent link="wheel" />
+<parent link="wheel0" />
 <child link="8x750roller_7" />
 <axis xyz="0 0 1"/>
@@ -317,5 +317,5 @@
 <joint name="roller_w0_7" type="continuous">
 <origin xyz="-0.0890001 -0.025494 0.0065875" rpy="1.5708 1.57079 0.174533" />
-<parent link="wheel" />
+<parent link="wheel0" />
 <child link="8x750roller_8" />
 <axis xyz="0 0 1"/>
@@ -350,5 +350,5 @@
 <joint name="roller_w0_8" type="continuous">
 <origin xyz="-0.0923522 0.00648329 0.0065875" rpy="1.5708 1.57079 -0.174533" />
-<parent link="wheel" />
+<parent link="wheel0" />
 <child link="8x750roller_9" />
 <axis xyz="0 0 1"/>
@@ -383,5 +383,5 @@
 <joint name="roller_w0_9" type="continuous">
 <origin xyz="-0.0845653 0.0376786 0.0065875" rpy="1.5708 1.57079 -0.523599" />
-<parent link="wheel" />
+<parent link="wheel0" />
 <child link="8x750roller_10" />
 <axis xyz="0 0 1"/>
@@ -416,5 +416,5 @@
 <joint name="roller_w0_10" type="continuous">
 <origin xyz="-0.0665785 0.0643294 0.0065875" rpy="2.44346 1.5708 0" />
-<parent link="wheel" />
+<parent link="wheel0" />
 <child link="8x750roller_11" />
 <axis xyz="0 0 1"/>
@@ -449,5 +449,5 @@
 <joint name="roller_w0_11" type="continuous">
 <origin xyz="-0.0405614 0.083221 0.0065875" rpy="2.79253 1.5708 0" />
-<parent link="wheel" />
+<parent link="wheel0" />
 <child link="8x750roller_12" />
 <axis xyz="0 0 1"/>
@@ -482,5 +482,5 @@
 <joint name="roller_w0_12" type="continuous">
 <origin xyz="-0.009652 0.092075 0.0065875" rpy="-1.5708 1.5708 1.5708" />
-<parent link="wheel" />
+<parent link="wheel0" />
 <child link="8x750roller_13" />
 <axis xyz="0 0 1"/>
@@ -515,5 +515,5 @@
 <joint name="roller_w0_13" type="continuous">
 <origin xyz="0.0224216 0.0898234 0.0065875" rpy="-1.5708 1.57079 1.22173" />
-<parent link="wheel" />
+<parent link="wheel0" />
 <child link="8x750roller_14" />
 <axis xyz="0 0 1"/>
@@ -548,5 +548,5 @@
 <joint name="roller_w0_14" type="continuous">
 <origin xyz="0.0517908 0.0767377 0.0065875" rpy="-1.5708 1.57079 0.872665" />
-<parent link="wheel" />
+<parent link="wheel0" />
 <child link="8x750roller_15" />
 <axis xyz="0 0 1"/>
@@ -581,5 +581,5 @@
 <joint name="roller_w0_15" type="continuous">
 <origin xyz="0.0749133 0.0543964 0.0065875" rpy="-1.5708 1.57079 0.523599" />
-<parent link="wheel" />
+<parent link="wheel0" />
 <child link="8x750roller_16" />
 <axis xyz="0 0 1"/>
@@ -614,5 +614,5 @@
 <joint name="roller_w0_16" type="continuous">
 <origin xyz="0.0890001 0.025494 0.0065875" rpy="-1.5708 1.57079 0.174533" />
-<parent link="wheel" />
+<parent link="wheel0" />
 <child link="8x750roller_17" />
 <axis xyz="0 0 1"/>
@@ -647,5 +647,5 @@
 <joint name="roller_w0_17" type="continuous">
 <origin xyz="0.0890001 -0.025494 0.0065875" rpy="1.5708 1.57079 -0.174533" />
-<parent link="wheel" />
+<parent link="wheel0" />
 <child link="8x750roller_18" />
 <axis xyz="0 0 1"/>
@@ -656,10 +656,10 @@
 <origin xyz="0.0076339 -0.242491 -0.130854" rpy="1.5708 1.50474e-12 2.69365e-06" />
 <parent link="body_link" />
-<child link="wheel" />
+<child link="wheel0" />
 <axis xyz="0 0 1"/>
 <limit effort="30" velocity="20" />
 <joint_properties friction="0.0"/>
 </joint>
-<link name="wheel_2">
+<link name="wheel1">
 <visual>
 <origin xyz="0.0157175 -0.000676884 -0.0110091" rpy="-1.5708 -7.59903e-17 5.39519e-23" />
@@ -713,5 +713,5 @@
 <joint name="roller_w1_0" type="continuous">
 <origin xyz="-0.0749133 0.0543964 -0.0015875" rpy="-1.5708 1.77409e-06 -0.523599" />
-<parent link="wheel_2" />
+<parent link="wheel1" />
 <child link="8x750roller_19" />
 <axis xyz="0 0 1"/>
@@ -746,5 +746,5 @@
 <joint name="roller_w1_1" type="continuous">
 <origin xyz="-0.0665785 0.0643294 -0.0015875" rpy="0.698132 -1.5708 0" />
-<parent link="wheel_2" />
+<parent link="wheel1" />
 <child link="8x750roller_20" />
 <axis xyz="0 0 1"/>
@@ -779,5 +779,5 @@
 <joint name="roller_w1_2" type="continuous">
 <origin xyz="-0.0405614 0.083221 -0.0015875" rpy="0.349066 -1.5708 0" />
-<parent link="wheel_2" />
+<parent link="wheel1" />
 <child link="8x750roller_21" />
 <axis xyz="0 0 1"/>
@@ -812,5 +812,5 @@
 <joint name="roller_w1_3" type="continuous">
 <origin xyz="-0.009652 0.092075 -0.0015875" rpy="-1.5708 -1.5708 1.5708" />
-<parent link="wheel_2" />
+<parent link="wheel1" />
 <child link="8x750roller_22" />
 <axis xyz="0 0 1"/>
@@ -845,5 +845,5 @@
 <joint name="roller_w1_4" type="continuous">
 <origin xyz="0.0224216 0.0898234 -0.0015875" rpy="-1.5708 -1.57079 1.22173" />
-<parent link="wheel_2" />
+<parent link="wheel1" />
 <child link="8x750roller_23" />
 <axis xyz="0 0 1"/>
@@ -878,5 +878,5 @@
 <joint name="roller_w1_5" type="continuous">
 <origin xyz="0.0517908 0.0767377 -0.0015875" rpy="-1.5708 -1.57079 0.872665" />
-<parent link="wheel_2" />
+<parent link="wheel1" />
 <child link="8x750roller_24" />
 <axis xyz="0 0 1"/>
@@ -911,5 +911,5 @@
 <joint name="roller_w1_6" type="continuous">
 <origin xyz="0.0749133 0.0543964 -0.0015875" rpy="-1.5708 2.89145e-06 0.523599" />
-<parent link="wheel_2" />
+<parent link="wheel1" />
 <child link="8x750roller_25" />
 <axis xyz="0 0 1"/>
@@ -944,5 +944,5 @@
 <joint name="roller_w1_7" type="continuous">
 <origin xyz="0.0890001 0.025494 -0.0015875" rpy="-1.5708 2.84675e-06 0.174533" />
-<parent link="wheel_2" />
+<parent link="wheel1" />
 <child link="8x750roller_26" />
 <axis xyz="0 0 1"/>
@@ -977,5 +977,5 @@
 <joint name="roller_w1_8" type="continuous">
 <origin xyz="0.0923522 -0.00648329 -0.0015875" rpy="-1.5708 2.4587e-06 -0.174533" />
-<parent link="wheel_2" />
+<parent link="wheel1" />
 <child link="8x750roller_27" />
 <axis xyz="0 0 1"/>
@@ -1010,5 +1010,5 @@
 <joint name="roller_w1_9" type="continuous">
 <origin xyz="0.0845653 -0.0376786 -0.0015875" rpy="-1.5708 1.77409e-06 -0.523599" />
-<parent link="wheel_2" />
+<parent link="wheel1" />
 <child link="8x750roller_28" />
 <axis xyz="0 0 1"/>
@@ -1043,5 +1043,5 @@
 <joint name="roller_w1_10" type="continuous">
 <origin xyz="0.0665785 -0.0643294 -0.0015875" rpy="-2.44346 -1.5708 0" />
-<parent link="wheel_2" />
+<parent link="wheel1" />
 <child link="8x750roller_29" />
 <axis xyz="0 0 1"/>
@@ -1076,5 +1076,5 @@
 <joint name="roller_w1_11" type="continuous">
 <origin xyz="0.0405614 -0.083221 -0.0015875" rpy="-2.79253 -1.5708 0" />
-<parent link="wheel_2" />
+<parent link="wheel1" />
 <child link="8x750roller_30" />
 <axis xyz="0 0 1"/>
@@ -1109,5 +1109,5 @@
 <joint name="roller_w1_12" type="continuous">
 <origin xyz="0.009652 -0.092075 -0.0015875" rpy="1.5708 -1.5708 1.5708" />
-<parent link="wheel_2" />
+<parent link="wheel1" />
 <child link="8x750roller_31" />
 <axis xyz="0 0 1"/>
@@ -1142,5 +1142,5 @@
 <joint name="roller_w1_13" type="continuous">
 <origin xyz="-0.0224216 -0.0898234 -0.0015875" rpy="1.5708 -1.57079 1.22173" />
-<parent link="wheel_2" />
+<parent link="wheel1" />
 <child link="8x750roller_32" />
 <axis xyz="0 0 1"/>
@@ -1175,5 +1175,5 @@
 <joint name="roller_w1_14" type="continuous">
 <origin xyz="-0.0517908 -0.0767377 -0.0015875" rpy="1.5708 -1.57079 0.872665" />
-<parent link="wheel_2" />
+<parent link="wheel1" />
 <child link="8x750roller_33" />
 <axis xyz="0 0 1"/>
@@ -1208,5 +1208,5 @@
 <joint name="roller_w1_15" type="continuous">
 <origin xyz="-0.0749133 -0.0543964 -0.0015875" rpy="1.5708 2.89145e-06 0.523599" />
-<parent link="wheel_2" />
+<parent link="wheel1" />
 <child link="8x750roller_34" />
 <axis xyz="0 0 1"/>
@@ -1241,5 +1241,5 @@
 <joint name="roller_w1_16" type="continuous">
 <origin xyz="-0.0890001 -0.025494 -0.0015875" rpy="1.5708 2.84675e-06 0.174533" />
-<parent link="wheel_2" />
+<parent link="wheel1" />
 <child link="8x750roller_35" />
 <axis xyz="0 0 1"/>
@@ -1274,5 +1274,5 @@
 <joint name="roller_w1_17" type="continuous">
 <origin xyz="-0.0923522 0.00648329 -0.0015875" rpy="1.5708 2.4587e-06 -0.174533" />
-<parent link="wheel_2" />
+<parent link="wheel1" />
 <child link="8x750roller_36" />
 <axis xyz="0 0 1"/>
@@ -1283,10 +1283,10 @@
 <origin xyz="-0.212654 0.132125 -0.130854" rpy="-1.5708 -1.50485e-12 1.0472" />
 <parent link="body_link" />
-<child link="wheel_2" />
+<child link="wheel1" />
 <axis xyz="0 0 1"/>
 <limit effort="30" velocity="20" />
 <joint_properties friction="0.0"/>
 </joint>
-<link name="wheel_3">
+<link name="wheel2">
 <visual>
 <origin xyz="0.0157175 -0.000676884 -0.0110091" rpy="-1.5708 1.21101e-16 3.64923e-22" />
@@ -1340,5 +1340,5 @@
 <joint name="roller_w2_0" type="continuous">
 <origin xyz="0.0890001 -0.025494 -0.0015875" rpy="-1.5708 -3.04078e-06 2.96706" />
-<parent link="wheel_3" />
+<parent link="wheel2" />
 <child link="8x750roller_37" />
 <axis xyz="0 0 1"/>
@@ -1373,5 +1373,5 @@
 <joint name="roller_w2_1" type="continuous">
 <origin xyz="0.0923522 0.00648329 -0.0015875" rpy="-1.5708 1.48959e-08 -2.96706" />
-<parent link="wheel_3" />
+<parent link="wheel2" />
 <child link="8x750roller_38" />
 <axis xyz="0 0 1"/>
@@ -1406,5 +1406,5 @@
 <joint name="roller_w2_2" type="continuous">
 <origin xyz="0.0845653 0.0376786 -0.0015875" rpy="-1.5708 -7.70262e-17 -2.61799" />
-<parent link="wheel_3" />
+<parent link="wheel2" />
 <child link="8x750roller_39" />
 <axis xyz="0 0 1"/>
@@ -1439,5 +1439,5 @@
 <joint name="roller_w2_3" type="continuous">
 <origin xyz="0.0665785 0.0643294 -0.0015875" rpy="2.44346 -1.5708 0" />
-<parent link="wheel_3" />
+<parent link="wheel2" />
 <child link="8x750roller_40" />
 <axis xyz="0 0 1"/>
@@ -1472,5 +1472,5 @@
 <joint name="roller_w2_4" type="continuous">
 <origin xyz="0.0405614 0.083221 -0.0015875" rpy="2.79253 -1.5708 0" />
-<parent link="wheel_3" />
+<parent link="wheel2" />
 <child link="8x750roller_41" />
 <axis xyz="0 0 1"/>
@@ -1505,5 +1505,5 @@
 <joint name="roller_w2_5" type="continuous">
 <origin xyz="0.009652 0.092075 -0.0015875" rpy="-3.14159 -1.5708 0" />
-<parent link="wheel_3" />
+<parent link="wheel2" />
 <child link="8x750roller_42" />
 <axis xyz="0 0 1"/>
@@ -1538,5 +1538,5 @@
 <joint name="roller_w2_6" type="continuous">
 <origin xyz="-0.0224216 0.0898234 -0.0015875" rpy="-2.79253 -1.5708 0" />
-<parent link="wheel_3" />
+<parent link="wheel2" />
 <child link="8x750roller_43" />
 <axis xyz="0 0 1"/>
@@ -1571,5 +1571,5 @@
 <joint name="roller_w2_7" type="continuous">
 <origin xyz="-0.0517908 0.0767377 -0.0015875" rpy="-2.44346 -1.5708 0" />
-<parent link="wheel_3" />
+<parent link="wheel2" />
 <child link="8x750roller_44" />
 <axis xyz="0 0 1"/>
@@ -1604,5 +1604,5 @@
 <joint name="roller_w2_8" type="continuous">
 <origin xyz="-0.0749133 0.0543964 -0.0015875" rpy="1.5708 -9.29494e-17 2.61799" />
-<parent link="wheel_3" />
+<parent link="wheel2" />
 <child link="8x750roller_45" />
 <axis xyz="0 0 1"/>
@@ -1637,5 +1637,5 @@
 <joint name="roller_w2_9" type="continuous">
 <origin xyz="-0.0890001 0.025494 -0.0015875" rpy="1.5708 -1.2854e-17 2.96706" />
-<parent link="wheel_3" />
+<parent link="wheel2" />
 <child link="8x750roller_46" />
 <axis xyz="0 0 1"/>
@@ -1670,5 +1670,5 @@
 <joint name="roller_w2_10" type="continuous">
 <origin xyz="-0.0923522 -0.00648329 -0.0015875" rpy="1.5708 -5.86296e-17 -2.96706" />
-<parent link="wheel_3" />
+<parent link="wheel2" />
 <child link="8x750roller_47" />
 <axis xyz="0 0 1"/>
@@ -1703,5 +1703,5 @@
 <joint name="roller_w2_11" type="continuous">
 <origin xyz="-0.0845653 -0.0376786 -0.0015875" rpy="1.5708 -7.70262e-17 -2.61799" />
-<parent link="wheel_3" />
+<parent link="wheel2" />
 <child link="8x750roller_48" />
 <axis xyz="0 0 1"/>
@@ -1736,5 +1736,5 @@
 <joint name="roller_w2_12" type="continuous">
 <origin xyz="-0.0665785 -0.0643294 -0.0015875" rpy="-0.698132 -1.5708 0" />
-<parent link="wheel_3" />
+<parent link="wheel2" />
 <child link="8x750roller_49" />
 <axis xyz="0 0 1"/>
@@ -1769,5 +1769,5 @@
 <joint name="roller_w2_13" type="continuous">
 <origin xyz="-0.0405614 -0.083221 -0.0015875" rpy="-0.349066 -1.5708 0" />
-<parent link="wheel_3" />
+<parent link="wheel2" />
 <child link="8x750roller_50" />
 <axis xyz="0 0 1"/>
@@ -1802,5 +1802,5 @@
 <joint name="roller_w2_14" type="continuous">
 <origin xyz="-0.009652 -0.092075 -0.0015875" rpy="7.41518e-14 -1.5708 0" />
-<parent link="wheel_3" />
+<parent link="wheel2" />
 <child link="8x750roller_51" />
 <axis xyz="0 0 1"/>
@@ -1835,5 +1835,5 @@
 <joint name="roller_w2_15" type="continuous">
 <origin xyz="0.0224216 -0.0898234 -0.0015875" rpy="0.349066 -1.5708 0" />
-<parent link="wheel_3" />
+<parent link="wheel2" />
 <child link="8x750roller_52" />
 <axis xyz="0 0 1"/>
@@ -1868,5 +1868,5 @@
 <joint name="roller_w2_16" type="continuous">
 <origin xyz="0.0517908 -0.0767377 -0.0015875" rpy="0.698132 -1.5708 0" />
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
Commit message: +y faces wheel2

File: urdf/urdf_generator/robot.urdf.xacro (robot description, xacro)
@@ -5,5 +5,5 @@
 </link>
 <joint name="body_joint" type="fixed">
-    <origin xyz="0 0 0" rpy="0 0 3.14"/>
+    <origin xyz="0 0 0" rpy="0 0 1.0472"/>
     <parent link="base_link"/>
     <child link="body_link"/>

Commit message: lidar and camera faces wheel2

File: urdf/urdf_generator/robot.urdf.xacro (robot description, xacro)
@@ -1929,6 +1929,6 @@
     </link>
     <joint name="lidar_mount_joint" type="fixed">
-        <origin xyz="0.0 -0.23 0.345" rpy="0.0 0.0 0.0"/>
-        <parent link="body_link"/>
+        <origin xyz="0.0 0.23 0.345" rpy="0.0 0.0 0.0"/>
+        <parent link="base_link"/>
         <child link="lidar_mount"/>
     </joint>
@@ -2033,6 +2033,6 @@
     <!-- Kinect Camera Joints -->
     <joint name="kinect_1_joint" type="fixed">
-        <origin xyz="-0.01239 -0.289682 0.28607" rpy="0 1.57 -1.57079632679"/>
-        <parent link="body_link"/>
+        <origin xyz="-0.01239 0.289682 0.28607" rpy="0 1.57 1.57079632679"/>
+        <parent link="base_link"/>
         <child link="kinect_1_link"/>
     </joint>
@@ -2060,5 +2060,5 @@
     <joint name="rplidar_joint" type="fixed">
         <axis xyz="0 1 0" />
-        <origin xyz="0 0 0" rpy="0 0 3.14159"/>
+        <origin xyz="0 0 0" rpy="0 0 -1.54"/>
         <parent link="lidar_mount"/>
         <child link="rplidar_link"/>

Commit message: lidar link name change rplidar_link -> lidar_link

File: urdf/urdf_generator/robot.urdf.xacro (robot description, xacro)
@@ -1934,5 +1934,5 @@
     </joint>
     <!-- Lidar Link -->
-  <link name="rplidar_link">
+  <link name="lidar_link">
     <collision>
       <origin xyz="0 0 0" rpy="1.5707 0 1.5707"/>
@@ -2062,5 +2062,5 @@
         <origin xyz="0 0 0" rpy="0 0 -1.54"/>
         <parent link="lidar_mount"/>
-        <child link="rplidar_link"/>
+        <child link="lidar_link"/>
     </joint>
 </robot>

Commit message: gazebo urdf deleted

File: urdf/urdf_generator/robot.urdf.xacro (robot description, xacro)
@@ -1,4 +1,16 @@
 <?xml version="1.1"?>
 <robot name="trikey" xmlns:xacro="http://ros.org/wiki/xacro">
+  <material name="black">
+    <color rgba="0. 0. 0. 1" />
+  </material>
+  <material name="dark_grey">
+    <color rgba="0.1 0.1 0.1 1" />
+  </material>
+  <material name="grey">
+    <color rgba="0.6 0.6 0.6 1" />
+  </material>
+  <material name="white">
+    <color rgba="0.9 0.9 0.9 1" />
+  </material>
 <xacro:include filename="$(find trikey_description)/urdf/urdf_generator/robot.gazebo.xacro" />
 <link name= "base_link">
@@ -1979,30 +1991,46 @@
         </inertial>
     </link>
-    <!-- Azure Kinect Camera Link (Bottom Camera) -->
-    <!-- <link name="kinect_2_link">
-        <visual>
-            <origin xyz="0 0 0" rpy="0 0 0"/>
-            <geometry>
-                <mesh filename="package://trikey_description/meshes/Azure_Kinect.stl"/>
-            </geometry>
-            <material name="kinect_material">
-                <color rgba="0.9 0.2 0.24 1.0"/>
-            </material>
-        </visual>
-        <collision>
-            <origin xyz="0.0 0.0 0.0"/>
-            <geometry>
-                <mesh filename="package://trikey_description/meshes/Azure_Kinect.stl"/>
-            </geometry>
-            <material name="kinect_material">
-                <color rgba="0.9 0.2 0.24 1.0"/>
-            </material>
-        </collision>
-        <inertial>
-            <origin xyz="0 0 0" rpy="0 0 0"/>
-            <mass value=".44" />
-            <inertia ixx="10.173985" ixy="0.212137"  ixz="-0.09591" iyy="5.191632" iyz="0.505713" izz="5.853716" />
-        </inertial>
-    </link> -->
+  <link name="camera_body">
+    <visual>
+      <origin xyz="0. 0. 0." />
+      <geometry>
+        <box size="0.0994 0.0996 0.023" />
+      </geometry>
+      <material name="white" />
+    </visual>
+  </link>
+  <link name="camera_base">
+    <visual>
+      <origin xyz="-0.013 0. 0." />
+      <geometry>
+        <box size="0.026 0.103 0.039" />
+      </geometry>
+      <material name="grey" />
+    </visual>
+  </link>
+  <link name="camera_visor">
+    <visual>
+      <origin xyz="-0.0128 0. 0." />
+      <geometry>
+        <box size="0.026 0.101 0.037" />
+      </geometry>
+      <material name="black" />
+    </visual>
+  </link>
+  <joint_name ="base_link_to_camera_base" type="fixed">
+    <parent link="base_link" />
+    <child link="camera_base" />
+    <origin xyz="-0.01239 0.289682 0.28607" rpy="0.0 0.0 1.57079632679" />
+  </joint>
+  <joint name="camera_base_to_body" type="fixed">
+    <parent link="camera_base" />
+    <child link="camera_body" />
+    <origin xyz="-0.0757 0. 0.008" rpy="0. 0. 0." />
+  </joint>
+  <joint name="camera_base_to_visor" type="fixed">
+    <parent link="camera_base" />
+    <child link="camera_visor" />
+    <origin xyz="0. 0. 0." rpy="0. 0. 0." />
+  </joint>
   <!-- Azure Kinect Camera Lense Link (Top Camera) -->
   <link name="kinect_1_lense_link">
@@ -2014,21 +2042,4 @@
     </visual>
   </link>
-  <!-- Azure Kinect Camera Lense Link (Bottom Camera) -->
-  <!-- <link name="kinect_2_lense_link">
-    <visual>
-      <origin xyz="0 0 0" rpy="0 1.57 0" />
-      <geometry>
-        <cylinder length="0.001" radius="0.01"/>
-      </geometry>
-    </visual>
-  </link>
-<link name="kinect_2_pcl_link">
-    <visual>
-      <origin xyz="0 0 0" rpy="0 0 0" />
-      <geometry>
-        <cylinder length="0.001" radius="0.01"/>
-      </geometry>
-    </visual>
-  </link> -->
     <!-- Kinect Camera Joints -->
     <joint name="kinect_1_joint" type="fixed">
@@ -2037,9 +2048,4 @@
         <child link="kinect_1_link"/>
     </joint>
-    <!-- <joint name="kinect_2_joint" type="fixed">
-        <origin xyz="0.01239 -0.289682 0.1734" rpy="0 2.0943951023931953 -1.57079632679"/>
-        <parent link="body_link"/>
-        <child link="kinect_2_link"/>
-    </joint> -->
     <joint name="kinect_1_lense_joint" type="fixed">
         <origin xyz="-0.03 0 0.01" rpy="3.14 -1.57 0"/>
@@ -2047,14 +2053,4 @@
         <child link="kinect_1_lense_link"/>
     </joint>
-    <!-- <joint name="kinect_2_lense_joint" type="fixed">
-        <origin xyz="-0.03 0 0.01" rpy="0 -1.57 0"/>
-        <parent link="kinect_2_link"/>
-        <child link="kinect_2_lense_link"/>
-    </joint>
-    <joint name="kinect_2_pcl_joint" type="fixed">
-        <origin xyz="0 0 0" rpy="0 0 -1.57079632679"/>
-        <parent link="kinect_2_link"/>
-        <child link="kinect_2_pcl_link"/>
-    </joint> -->
     <!-- Lidar Joint -->
     <joint name="rplidar_joint" type="fixed">

Commit message: kinect link added to match acutal link names

File: urdf/urdf_generator/robot.urdf.xacro (robot description, xacro)
@@ -2018,8 +2018,8 @@
     </visual>
   </link>
-  <joint_name ="base_link_to_camera_base" type="fixed">
-    <parent link="base_link" />
-    <child link="camera_base" />
-    <origin xyz="-0.01239 0.289682 0.28607" rpy="0.0 0.0 1.57079632679" />
+  <joint name="base_link_to_camera_base" type="fixed">
+      <origin xyz="-0.01239 0.289682 0.28607" rpy="-1.57 0.0 1.57079632679" />
+      <parent link="base_link" />
+      <child link="camera_base" />
   </joint>
   <joint name="camera_base_to_body" type="fixed">

Commit message: lidar yaw fixed to face +x

File: urdf/urdf_generator/robot.urdf.xacro (robot description, xacro)
@@ -2056,5 +2056,5 @@
     <joint name="rplidar_joint" type="fixed">
         <axis xyz="0 1 0" />
-        <origin xyz="0 0 0" rpy="0 0 -1.54"/>
+        <origin xyz="0 0 0" rpy="0 0 0"/>
         <parent link="lidar_mount"/>
         <child link="lidar_link"/>

Commit message: lidar +x fix

File: urdf/urdf_generator/robot.urdf.xacro (robot description, xacro)
@@ -2056,5 +2056,5 @@
     <joint name="rplidar_joint" type="fixed">
         <axis xyz="0 1 0" />
-        <origin xyz="0 0 0" rpy="0 0 0"/>
+        <origin xyz="0 0 0" rpy="0 0 3.14"/>
         <parent link="lidar_mount"/>
         <child link="lidar_link"/>
